File: parallel-led.kicad_pcb (KiCad board)
At the start: 2 copper layers, 97 x 98 mm, 11 parts

Commit message: add + - sign for each led
Other:
- board text added: "+"
- board text added: "-"
Changed lines of the file:
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@@
   (gr_rect (start 63 51) (end 160 149)
     (stroke (width 0.1) (type default)) (fill none) (layer "Edge.Cuts"))
+  (gr_text "+" (at 135.1 135.8) (layer "F.SilkS")
+    (effects (font (size 1.5 1.5) (thickness 0.3) bold) (justify left bottom))
+  )
+  (gr_text "-" (at 144.1 135.7) (layer "F.SilkS")
+    (effects (font (size 1.5 1.5) (thickness 0.3) bold) (justify left bottom))
+  )
   (gr_text "B+" (at 77 109) (layer "F.SilkS")
     (effects (font (size 1.25 1.25) (thickness 0.2)) (justify left bottom))
+  )
+  (gr_text "-" (at 144.1 74.7) (layer "F.SilkS")
+    (effects (font (size 1.5 1.5) (thickness 0.3) bold) (justify left bottom))
+  )
+  (gr_text "+" (at 135.1 104.8) (layer "F.SilkS")
+    (effects (font (size 1.5 1.5) (thickness 0.3) bold) (justify left bottom))
+  )
+  (gr_text "-" (at 144.1 104.7) (layer "F.SilkS")
+    (effects (font (size 1.5 1.5) (thickness 0.3) bold) (justify left bottom))
+  )
+  (gr_text "-" (at 144.1 120.7) (layer "F.SilkS")
+    (effects (font (size 1.5 1.5) (thickness 0.3) bold) (justify left bottom))
+  )
+  (gr_text "+" (at 135.1 89.95) (layer "F.SilkS")
+    (effects (font (size 1.5 1.5) (thickness 0.3) bold) (justify left bottom))
+  )
+  (gr_text "+" (at 135.1 74.7) (layer "F.SilkS")
+    (effects (font (size 1.5 1.5) (thickness 0.3) bold) (justify left bottom))
   )
   (gr_text "B-" (at 77 95) (layer "F.SilkS")
     (effects (font (size 1.25 1.25) (thickness 0.2)) (justify left bottom))
   )
+  (gr_text "+" (at 135.1 120.8) (layer "F.SilkS")
+    (effects (font (size 1.5 1.5) (thickness 0.3) bold) (justify left bottom))
+  )
+  (gr_text "-" (at 144.1 89.7) (layer "F.SilkS")
+    (effects (font (size 1.5 1.5) (thickness 0.3) bold) (justify left bottom))
+  )
   (segment (start 94 120) (end 94 89) (width 0.25) (layer "F.Cu") (net 1))

Commit message: modify D1; modify battery
Other:
- board text removed: "+"
- board text removed: "-"
- board text removed: "B+"
- board text removed: "B-"
Changed lines of the file:
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@@
         (effects (font (size 1 1) (thickness 0.15)))
+    )
+    (fp_text user "-" (at -3.9 0.7 180 unlocked) (layer "F.SilkS")
+        (effects (font (size 1.25 1.25) (thickness 0.15)) (justify left bottom))
+    )
+    (fp_text user "+" (at 4.7 0.7 180 unlocked) (layer "F.SilkS")
+        (effects (font (size 1.25 1.25) (thickness 0.15)) (justify left bottom))
     )
     (fp_text user "${REFERENCE}" (at 1.25 0) (layer "F.Fab")
@@
     )
     (fp_line (start -1.29 -1.545) (end -1.29 1.545)
+      (stroke (width 0.12) (type solid)) (layer "F.SilkS"))
+    (fp_line (start -1.29 0) (end 4.26 -0.000462)
+      (stroke (width 0.12) (type default)) (layer "F.SilkS"))
+    (fp_line (start -1.26 0) (end 2.9 -2.4)
+      (stroke (width 0.12) (type solid)) (layer "F.SilkS"))
+    (fp_line (start -1.23 0) (end -1.29 0)
+      (stroke (width 0.1) (type default)) (layer "F.SilkS"))
+    (fp_line (start 2.9 -2.4) (end 2.9 2.5)
+      (stroke (width 0.12) (type solid)) (layer "F.SilkS"))
+    (fp_line (start 2.9 2.5) (end -1.26 0)
       (stroke (width 0.12) (type solid)) (layer "F.SilkS"))
     (fp_arc (start -1.29 -1.54483) (mid 2.072002 -2.880433) (end 4.26 0.000462)
@@
         (effects (font (size 1.25 1.25) (thickness 0.2)))
     )
-    (fp_text value "3V" (at 3 8.54 90) (layer "F.Fab")
-        (effects (font (size 1 1) (thickness 0.15)))
+    (fp_text value "3V" (at 3 8.54 90) (layer "F.Fab") hide
+        (effects (font (size 1 1) (thickness 0.15)))
+    )
+    (fp_text user "B-" (at 8.9 -0.66 unlocked) (layer "F.SilkS")
+        (effects (font (size 1.25 1.25) (thickness 0.15)) (justify left bottom))
+    )
+    (fp_text user "B+" (at -4.5 -0.66 unlocked) (layer "F.SilkS")
+        (effects (font (size 1.25 1.25) (thickness 0.15)) (justify left bottom))
     )
     (fp_text user "${REFERENCE}" (at 2.5 -2 90) (layer "F.Fab")
@@
   (gr_rect (start 63 51) (end 160 149)
     (stroke (width 0.1) (type default)) (fill none) (layer "Edge.Cuts"))
-  (gr_text "+" (at 135.1 135.8) (layer "F.SilkS")
-    (effects (font (size 1.5 1.5) (thickness 0.3) bold) (justify left bottom))
-  )
-  (gr_text "-" (at 144.1 135.7) (layer "F.SilkS")
-    (effects (font (size 1.5 1.5) (thickness 0.3) bold) (justify left bottom))
-  )
-  (gr_text "B+" (at 77 109) (layer "F.SilkS")
-    (effects (font (size 1.25 1.25) (thickness 0.2)) (justify left bottom))
-  )
-  (gr_text "-" (at 144.1 74.7) (layer "F.SilkS")
-    (effects (font (size 1.5 1.5) (thickness 0.3) bold) (justify left bottom))
-  )
-  (gr_text "+" (at 135.1 104.8) (layer "F.SilkS")
-    (effects (font (size 1.5 1.5) (thickness 0.3) bold) (justify left bottom))
-  )
-  (gr_text "-" (at 144.1 104.7) (layer "F.SilkS")
-    (effects (font (size 1.5 1.5) (thickness 0.3) bold) (justify left bottom))
-  )
-  (gr_text "-" (at 144.1 120.7) (layer "F.SilkS")
-    (effects (font (size 1.5 1.5) (thickness 0.3) bold) (justify left bottom))
-  )
-  (gr_text "+" (at 135.1 89.95) (layer "F.SilkS")
-    (effects (font (size 1.5 1.5) (thickness 0.3) bold) (justify left bottom))
-  )
-  (gr_text "+" (at 135.1 74.7) (layer "F.SilkS")
-    (effects (font (size 1.5 1.5) (thickness 0.3) bold) (justify left bottom))
-  )
-  (gr_text "B-" (at 77 95) (layer "F.SilkS")
-    (effects (font (size 1.25 1.25) (thickness 0.2)) (justify left bottom))
-  )
-  (gr_text "+" (at 135.1 120.8) (layer "F.SilkS")
-    (effects (font (size 1.5 1.5) (thickness 0.3) bold) (justify left bottom))
-  )
-  (gr_text "-" (at 144.1 89.7) (layer "F.SilkS")
-    (effects (font (size 1.5 1.5) (thickness 0.3) bold) (justify left bottom))
-  )
   (segment (start 94 120) (end 94 89) (width 0.25) (layer "F.Cu") (net 1))
   (segment (start 94 135) (end 94 120) (width 0.25) (layer "F.Cu") (net 1))
